Commit message: update laser and adding base_footprint frame

File: searcherbot_description/urdf/colors.urdf.xacro (robot description, xacro)
@@ -18,4 +18,5 @@
   <xacro:create_color name="Red" value="1 0 0 1"/>
   <xacro:create_color name="BlueGlow" value="0.5 0.5 0.5 1"/>
+  <xacro:create_color name="Yellow" value="1 1 0 1"/>
   <xacro:gazebo_color link="base_link" color="BlueGlow"/>
   <xacro:gazebo_color link="camera_link" color="Black"/>
@@ -24,3 +25,4 @@
   <xacro:gazebo_color link="right_wheel_link" color="DarkGrey"/>
   <xacro:gazebo_color link="support_link" color="Grey"/>
+  <xacro:gazebo_color link="support_link2" color="Yellow"/>
 </robot>

File: searcherbot_description/urdf/searcherbot.urdf (robot description, URDF)
Before this commit: robot searcherbot, 6 links, 5 joints
Links:
- added link base_footprint, mass 0.0001; visual box size=0.001 0.001 0.001
- added link support_link2, mass 3.0; collision sphere radius=0.125; visual sphere radius=0.125
Joints:
- added joint base_footprint_joint: type fixed, parent base_footprint, child base_link, origin xyz=0 0 0.3 rpy=0 0 0
- added joint support_joint2: type continuous, parent base_link, child support_link2, origin xyz=-0.15 0 -0.175 rpy=-1.5708 0 0, axis 0 0 1.0, limit effort=0 velocity=0
- joint left_wheel_joint: limit effort=1000.0 velocity=5.0 -> effort=100.0 velocity=5.0
- joint right_wheel_joint: limit effort=1000.0 velocity=5.0 -> effort=100.0 velocity=5.0

File: searcherbot_description/urdf/searcherbot.xacro (robot description, xacro)
@@ -5,4 +5,32 @@
   <xacro:include filename="$(find searcherbot_description)/urdf/sensors/laser.urdf.xacro"/>
   <xacro:include filename="$(find searcherbot_description)/urdf/sensors/camera.urdf.xacro"/>
+  <xacro:macro name="set_transmission" params="joint_name">
+    <transmission name="${joint_name}_trans">
+      <type>transmission_interface/SimpleTransmission</type>
+      <joint name="${joint_name}"/>
+      <actuator naem="${joint_name}_motor">
+        <hardwareInterface>EffortJointInterface</hardwareInterface>
+        <mechanicalReduction>1.0</mechanicalReduction>
+      </actuator>
+    </transmission>
+  </xacro:macro>
+  <link name="base_footprint">
+    <inertial>
+      <mass value="0.0001" />
+      <origin xyz="0 0 0" />
+      <inertia ixx="0.0001" ixy="0.0" ixz="0.0"
+          iyy="0.0001" iyz="0.0"
+          izz="0.0001" />
+    </inertial>
+    <visual>
+        <origin xyz="0 0 0" rpy="0 0 0" />
+        <geometry>
+            <box size="0.001 0.001 0.001" />
+        </geometry>
+    </visual>
+  </link>
+  <gazebo reference="base_footprint">
+    <turnGravityOff>false</turnGravityOff>
+  </gazebo>
   <link name="base_link">
     <inertial>
@@ -125,4 +153,29 @@
     </collision>
   </link>
+  <link name="support_link2">
+    <inertial>
+      <origin xyz="0 0 0" rpy="0 0 0"/>
+      <mass value="3.0"/>
+      <inertia ixx="0.00625" ixy="0" ixz="0" iyy="0.00625" iyz="0" izz="0.00625"/>
+    </inertial>
+    <visual>
+      <origin xyz="0 0 0" rpy="1.5708 0 0"/>
+      <geometry>
+        <sphere radius="0.125"/>
+      </geometry>
+      <material name="Yellow"/>
+    </visual>
+    <collision name="support2">
+      <origin xyz="0 0 0" rpy="1.5708 0 0"/>
+      <geometry>
+        <sphere radius="0.125"/>
+      </geometry>
+    </collision>
+  </link>
+  <joint name="base_footprint_joint" type="fixed">
+    <origin xyz="0 0 0.3" rpy="0 0 0" />
+    <parent link="base_footprint"/>
+    <child link="base_link" />
+  </joint>
   <joint name="camera_joint" type="fixed">
     <origin xyz="0.225 0 0.225" rpy="0 0 0"/>
@@ -140,5 +193,5 @@
     <child link="left_wheel_link"/>
     <axis xyz="0 0 1.0"/>
-    <limit effort="1000.0" velocity="5.0"/>
+    <limit effort="100.0" velocity="5.0"/>
   </joint>
   <joint name="right_wheel_joint" type="continuous">
@@ -147,5 +200,5 @@
     <child link="right_wheel_link"/>
     <axis xyz="0 0 1.0"/>
-    <limit effort="1000.0" velocity="5.0"/>
+    <limit effort="100.0" velocity="5.0"/>
   </joint>
   <joint name="support_joint" type="continuous">
@@ -156,4 +209,13 @@
     <limit effort="0" velocity="0"/>
   </joint>
+  <joint name="support_joint2" type="continuous">
+    <origin xyz="-0.15 0 -0.175" rpy="-1.5708 0 0"/>
+    <parent link="base_link"/>
+    <child link="support_link2"/>
+    <axis xyz="0 0 1.0"/>
+    <limit effort="0" velocity="0"/>
+  </joint>
+  <xacro:set_transmission joint_name="left_wheel_joint"/>
+  <xacro:set_transmission joint_name="right_wheel_joint"/>
   <!-- Adding Sensors -->
   <xacro:set_laser reference_frame="laser_link"/>
@@ -180,5 +242,5 @@
       <odometryFrame>odom</odometryFrame>
       <odometryTopic>odom</odometryTopic>
-      <robotBaseFrame>base_link</robotBaseFrame>
+      <robotBaseFrame>base_footprint</robotBaseFrame>
     </plugin>
   </gazebo>

File: searcherbot_description/urdf/sensors/laser.urdf.xacro (robot description, xacro)
@@ -5,5 +5,5 @@
     <gazebo reference="${reference_frame}">
       <turnGravityOff>false</turnGravityOff>
-      <sensor type="ray" name="laser360_sensor">
+      <sensor type="ray" name="laser180_sensor">
         <pose>0 0 0 0 0 0</pose>
         <visualize>false</visualize>
@@ -14,6 +14,6 @@
               <samples>720</samples>
               <resolution>1</resolution>
-              <min_angle>-3.14</min_angle>
-              <max_angle>3.14</max_angle>
+              <min_angle>-1.57</min_angle>
+              <max_angle>1.57</max_angle>
             </horizontal>
           </scan>
